File: 8ch-mosfet/8ch-mosfet.kicad_pcb (KiCad board)
At the start: 2 copper layers, 184.5 x 137 mm, 204 parts, among them J10 Screw_Terminal_01x02, J11 Screw_Terminal_01x02, J12 Screw_Terminal_01x02, J13 I2C, J14 N2K, J3 Screw_Terminal_01x08, J5 Screw_Terminal_01x02, J6 Screw_Terminal_01x02, J7 Screw_Terminal_01x02, J8 Screw_Terminal_01x02, J9 Screw_Terminal_01x02, M1 Fan_4pin, M2 Fan_4pin, Q1 2N7002, Q10 IPB110P06LM, Q11 2N7002, Q12 IPB110P06LM, Q13 2N7002, Q14 IPB110P06LM, Q15 2N7002, Q16 IPB110P06LM, Q2 IPB110P06LM, Q21 BC846, Q22 BC856, Q23 BC846, Q24 BC856, Q25 BC846, Q26 BC856, Q27 BC846, Q28 BC856, Q29 BC846, Q3 2N7002, Q30 BC856, Q31 BC846, Q32 BC856, Q33 BC846, Q34 BC856, Q35 BC846, Q36 BC856, Q4 IPB110P06LM, Q5 2N7002, Q6 IPB110P06LM, Q7 2N7002, Q8 IPB110P06LM, Q9 2N7002, U1 ESP32-DEVKITC, U10 ACS725xLCTR-20AU, U11 ACS725xLCTR-20AU, U12 ACS725xLCTR-20AU, U13 MCP1502-33, U15 MCP3425A0T-ECH, U2 MCP3208, U4 XL1509-5.0, U5 ACS725xLCTR-20AU, U6 ACS725xLCTR-20AU, U7 ACS725xLCTR-20AU, U8 ACS725xLCTR-20AU, U9 ACS725xLCTR-20AU

Commit message: more progress on new 8ch board.
Parts:
- removed J11, J12: Screw_Terminal_01x02, yarrboard:Molex 1x02 .375
- removed U2: MCP3208, Package_SO:SOIC-16_3.9x9.9mm_P1.27mm
- added J1: Conn_01x01, yarrboard:T44001, F.Cu at (-24.5, 84.4)
- added J2: Conn_01x01, yarrboard:T44001, F.Cu at (24.3, 74.3)
- added JP2: SolderJumper_2_Open, Jumper:SolderJumper-2_P1.3mm_Open_RoundedPad1.0x1.5mm, F.Cu at (-17.7, 70.5)
- added JP3: SolderJumper_2_Open, Jumper:SolderJumper-2_P1.3mm_Open_RoundedPad1.0x1.5mm, F.Cu at (-17.7, 74.0)
- added Q17: 2N7002, Package_TO_SOT_SMD:SOT-23, F.Cu at (29.1, 84.3)
- added Q18: 2N7002, Package_TO_SOT_SMD:SOT-23, F.Cu at (22.2, 84.3)
- added R44: 1k, Resistor_SMD:R_0805_2012Metric_Pad1.20x1.40mm_HandSolder, F.Cu at (22.1, 88.0)
- added U3: MCP3564R, Package_SO:TSSOP-20_4.4x6.5mm_P0.65mm, F.Cu at (-24.3, 72.7)
- F9: value mSMD050-60V -> mSMD050-60V
- J10, J5, J6, J7, J8, J9: value Screw_Terminal_01x02 -> Conn_01x01; footprint yarrboard:Molex 1x02 .375 -> yarrboard:T44001
- R43: value 0R -> 1k
- U1: value ESP32-DEVKITC -> ~; footprint yarrboard:ESP32-DevKitC -> yarrboard:Waveshare-ESP32-S3-dev-kit
- moved J10 176.6 mm to (13.2, 87.5)
- moved J9 172.5 mm to (2.08, 74.3)
- moved J8 161.2 mm to (-9.02, 87.5)
- moved J7 126.6 mm to (13.2, 74.3)
- moved J6 114.2 mm to (2.08, 87.5)
- moved J5 112.3 mm to (-9.02, 74.3)
- moved U1 104.9 mm to (-28.3, 40.6)
- moved R43 73.9 mm to (29.0, 88.0), turned to 0 degrees
- renumbered locked to J4
Connections:
- C49 pad 1: REF_3V3 -> +3.3V
- C49 pad 2: GNDA -> GNDD
- F1 pad 3: Net-(Q2-D) -> Net-(D10-K)
- F2 pad 3: Net-(Q4-D) -> Net-(D11-K)
- F3 pad 3: Net-(Q6-D) -> Net-(D12-K)
- F4 pad 3: Net-(Q8-D) -> Net-(D13-K)
- F5 pad 3: Net-(Q10-D) -> Net-(D14-K)
- F6 pad 3: Net-(Q12-D) -> Net-(D15-K)
- F7 pad 3: Net-(Q14-D) -> Net-(D16-K)
- F8 pad 3: Net-(Q16-D) -> Net-(D17-K)
- J10 pad 1: Net-(D15-K) -> Net-(D17-K)
- J5 pad 1: Net-(D10-K) -> Net-(D12-K)
- J6 pad 1: Net-(D11-K) -> Net-(D13-K)
- J7 pad 1: Net-(D12-K) -> Net-(D14-K)
- J8 pad 1: Net-(D13-K) -> Net-(D15-K)
- J9 pad 1: Net-(D14-K) -> Net-(D16-K)
- M1 pad 1: GNDD -> Net-(M1--)
- M2 pad 1: GNDD -> Net-(M2--)
- R43 pad 1: Net-(U1-GPIO15) -> Net-(Q17-G)
- R43 pad 2: FAN_TACH2 -> FAN_MOSFET1
- U1 pad 10: /CHANNEL 3/PWM -> CAN_TX
- U1 pad 11: /CHANNEL 4/PWM -> CAN_RX
- U1 pad 12: /CHANNEL 5/PWM -> SDA
- U1 pad 13: /CHANNEL 6/PWM -> unconnected-(U1-GPIO3-Pad13)
- U1 pad 14: GNDD -> unconnected-(U1-GPIO46-Pad14)
- U1 pad 15: /CHANNEL 7/PWM -> SCL
- U1 pad 16: unconnected-(U1-GPIO9-Pad16) -> SS
- U1 pad 17: unconnected-(U1-GPIO10-Pad17) -> MOSI
- U1 pad 18: unconnected-(U1-GPIO11-Pad18) -> SCK
- U1 pad 19: ESP32_5V -> MISO
- U1 pad 2: unconnected-(U1-EN-Pad2) -> +3.3V
- U1 pad 21: unconnected-(U1-GPIO7-Pad21) -> ESP32_5V
- U1 pad 22: unconnected-(U1-GPIO8-Pad22) -> GNDD
- U1 pad 23: Net-(U1-GPIO15) -> GNDD
- U1 pad 24: FAN_PWM2 -> GNDD
- U1 pad 26: CAN_RX -> unconnected-(U1-USB_D+-Pad26)
- U1 pad 27: FAN_PWM1 -> FAN_TACH1
- U1 pad 28: SS -> FAN_PWM1
- U1 pad 29: CAN_TX -> FAN_MOSFET1
- U1 pad 30: SCK -> unconnected-(U1-GPIO45-Pad30)
- U1 pad 31: MISO -> unconnected-(U1-GPIO0-Pad31)
- U1 pad 32: GNDD -> unconnected-(U1-GPIO35-Pad32)
- U1 pad 33: SDA -> /CHANNEL 7/PWM
- U1 pad 34: unconnected-(U1-GPIO3-Pad34) -> /CHANNEL 6/PWM
- U1 pad 36: SCL -> /CHANNEL 5/PWM
- U1 pad 37: MOSI -> /CHANNEL 4/PWM
- U1 pad 38: GNDD -> /CHANNEL 3/PWM
- U1 pad 4: FAN_TACH1 -> unconnected-(U1-GPIO4-Pad4)
- U1 pad 5: unconnected-(U1-GPIO34-Pad5) -> FAN_MOSFET2
- U1 pad 6: unconnected-(U1-GPIO35-Pad6) -> FAN_PWM2
- U1 pad 7: /CHANNEL 0/PWM -> FAN_TACH2
- U1 pad 8: /CHANNEL 1/PWM -> unconnected-(U1-GPIO15-Pad8)
- U1 pad 9: /CHANNEL 2/PWM -> unconnected-(U1-GPIO16-Pad9)
Routing:
- net unconnected-(J13-MountPin-PadMP)_1: track 5.60 -> 0.00 mm
- net unconnected-(J13-MountPin-PadMP): track 0.00 -> 5.60 mm
- net Net-(U1-GPIO15): track 2.96 -> 0.00 mm
- net (no net): track 0.00 -> 2.96 mm
- net GNDD: track 114.6 -> 117.3 mm
- net GNDA: track 16.3 -> 13.6 mm
Other:
- board text added: "CH0+"
- board text added: "CH0-"
- board text added: "CH1+"
- board text added: "CH1-"
- board text added: "CH2+"
- board text added: "CH2-"
- board text added: "CH3+"
- board text added: "CH3-"
- board text added: "CH4+"
- board text added: "CH4-"
- board text added: "CH5+"
- board text added: "CH5-"
- board text added: "CH6+"
- board text added: "CH6-"
- board text added: "CH7+"
- board text added: "CH7-"
- board text removed: "locked"

Commit message: new design is going to be sick.
Parts:
- moved U1 141.1 mm to (54.2, 155.1), turned to 90 degrees
- moved J1 120.5 mm to (88.0, 127.5)
- moved J2 34.0 mm to (20.5, 40.5)
- moved H5 28.0 mm to (231.5, 131.5)
- moved H1 20.7 mm to (53.0, 152.0)
- moved H2 10.5 mm to (53.0, 86.0)
- moved J4 4.23 mm to (252.1, 145.0)
Routing:
- net Net-(Q2-D): vias 48 -> 0
Other:
- copper layers 2 -> 4

Commit message: updated busbar design.
Parts:
- J3, J4: footprint yarrboard:Busbar 1x9 .375in -> yarrboard:Busbar Rev D
- moved J3 168.3 mm to (88.0, 28.0), turned to 0 degrees
- moved J4 165.6 mm to (86.5, 147.0), turned to 0 degrees
- moved D10 12.7 mm to (86.5, 129.6)
- moved J1 5.72 mm to (86.5, 122.0), turned to 180 degrees
- moved C4 5.43 mm to (90.4, 107.0)
- moved R47 5.43 mm to (90.4, 109.3)
- moved C3 5.43 mm to (90.4, 113.9)
- moved C5 5.43 mm to (90.4, 111.6)
- moved U5 5.08 mm to (84.4, 111.2)
- moved Q2 2.23 mm to (86.5, 98.5)
Routing:
- net +3.3V: track 376.8 -> 159.5 mm, vias 12 -> 0
- net /ADC/A7: track 170.9 -> 0.00 mm, vias 2 -> 0
- net Net-(D10-K): track 0.00 -> 166.1 mm
- net ESP32_5V: track 167.7 -> 14.0 mm, vias 2 -> 0
- net GNDPWR: track 131.2 -> 0.00 mm
- net FAN_PWM2: track 130.0 -> 3.56 mm, vias 2 -> 0
- net FAN_PWM1: track 113.4 -> 5.09 mm, vias 2 -> 0
- net FAN_TACH2: track 123.0 -> 20.3 mm, vias 2 -> 0
- net CAN_RX: track 107.6 -> 16.8 mm, vias 2 -> 0
- net /CHANNEL 7/PWM: track 241.3 -> 156.0 mm, vias 2 -> 0
- net SCL: track 81.6 -> 0.00 mm, vias 4 -> 0
- net /CHANNEL 6/PWM: track 216.7 -> 136.4 mm, vias 2 -> 0
- net CAN_TX: track 104.0 -> 24.2 mm, vias 3 -> 0
- net GNDD: track 117.3 -> 38.0 mm, vias 44 -> 0
- net /CHANNEL 5/PWM: track 194.8 -> 116.9 mm, vias 2 -> 0
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
Commit message: big update - 12ch, volt adc, senders, etc.
Parts:
- removed the C30 at (67.6, 102.1)
- removed the D29 at (58.0, 73.5)
- removed the D30 at (58.0, 69.4)
- removed the D31 at (58.0, 65.4)
- removed the JP1 at (72.3, 104.3)
- removed LOGO: Logo Small, yarrboard:Logo Small
- removed the U13 at (72.3, 100.8)
- added C26: 100nF, Capacitor_SMD:C_0805_2012Metric_Pad1.18x1.45mm_HandSolder, F.Cu at (-53.8, 31.2)
- added C31: 100nF, Capacitor_SMD:C_0805_2012Metric_Pad1.18x1.45mm_HandSolder, F.Cu at (-53.8, 40.2)
- added C36: 100nF, Capacitor_SMD:C_0805_2012Metric_Pad1.18x1.45mm_HandSolder, F.Cu at (-37.1, 39.2)
- added C37: 1nF, Capacitor_SMD:C_0805_2012Metric_Pad1.18x1.45mm_HandSolder, F.Cu at (-60.6, -28.6)
- added C38: 100nF, Capacitor_SMD:C_0805_2012Metric_Pad1.18x1.45mm_HandSolder, F.Cu at (-60.6, -25.6)
- added C39: 4.7nF, Capacitor_SMD:C_0805_2012Metric_Pad1.18x1.45mm_HandSolder, F.Cu at (-60.6, -22.6)
- added C40: 1nF, Capacitor_SMD:C_0805_2012Metric_Pad1.18x1.45mm_HandSolder, F.Cu at (-26.5, 5.63)
- added C41: 100nF, Capacitor_SMD:C_0805_2012Metric_Pad1.18x1.45mm_HandSolder, F.Cu at (-26.5, 8.64)
- added C42: 4.7nF, Capacitor_SMD:C_0805_2012Metric_Pad1.18x1.45mm_HandSolder, F.Cu at (-26.5, 11.7)
- added C43: 1nF, Capacitor_SMD:C_0805_2012Metric_Pad1.18x1.45mm_HandSolder, F.Cu at (-60.6, 5.63)
- added C44: 100nF, Capacitor_SMD:C_0805_2012Metric_Pad1.18x1.45mm_HandSolder, F.Cu at (-60.6, 8.64)
- added C45: 4.7nF, Capacitor_SMD:C_0805_2012Metric_Pad1.18x1.45mm_HandSolder, F.Cu at (-60.6, 11.7)
- added C46: 1nF, Capacitor_SMD:C_0805_2012Metric_Pad1.18x1.45mm_HandSolder, F.Cu at (-26.5, -28.6)
- added C47: 100nF, Capacitor_SMD:C_0805_2012Metric_Pad1.18x1.45mm_HandSolder, F.Cu at (-26.5, -25.6)
- added C49: 100nF, Capacitor_SMD:C_0805_2012Metric_Pad1.18x1.45mm_HandSolder, F.Cu at (-19.7, 1.56)
- added C50: 100nF, Capacitor_SMD:C_0805_2012Metric_Pad1.18x1.45mm_HandSolder, F.Cu at (-21.6, 35.8)
- added C51: 100nF, Capacitor_SMD:C_0805_2012Metric_Pad1.18x1.45mm_HandSolder, F.Cu at (-19.7, 11.2)
- added D34: BAT54S, Package_TO_SOT_SMD:SOT-23, F.Cu at (-49.0, 41.3)
- added D37: LED, LED_SMD:LED_0805_2012Metric_Pad1.15x1.40mm_HandSolder, F.Cu at (-78.9, -8.78)
- added D38: 15V, Diode_SMD:D_SOD-323_HandSoldering, F.Cu at (-78.7, -11.8)
- added D40: LED, LED_SMD:LED_0805_2012Metric_Pad1.15x1.40mm_HandSolder, F.Cu at (-44.7, 25.5)
- added D41: 15V, Diode_SMD:D_SOD-323_HandSoldering, F.Cu at (-44.6, 22.5)
- added D42: SS16, Diode_SMD:D_SMA, F.Cu at (-43.1, 18.8)
- added D43: LED, LED_SMD:LED_0805_2012Metric_Pad1.15x1.40mm_HandSolder, F.Cu at (-78.9, 25.5)
- added D44: 15V, Diode_SMD:D_SOD-323_HandSoldering, F.Cu at (-78.7, 22.5)
- added D45: SS16, Diode_SMD:D_SMA, F.Cu at (-77.2, 18.8)
- added D46: LED, LED_SMD:LED_0805_2012Metric_Pad1.15x1.40mm_HandSolder, F.Cu at (-44.7, -8.78)
- added D47: 15V, Diode_SMD:D_SOD-323_HandSoldering, F.Cu at (-44.6, -11.8)
- added D48: SS16, Diode_SMD:D_SMA, F.Cu at (-43.1, -15.5)
- added F11: 25A, yarrboard:ATC Bypass Fuse, F.Cu at (-75.3, -34.5)
- added F12: 25A, yarrboard:ATC Bypass Fuse, F.Cu at (-41.2, -0.23)
- added F13: 25A, yarrboard:ATC Bypass Fuse, F.Cu at (-75.3, -0.23)
- added F14: 25A, yarrboard:ATC Bypass Fuse, F.Cu at (-41.2, -34.5)
- added J12: Conn_01x01, yarrboard:T44001, F.Cu at (-85.8, -12.2)
- added J13: Conn_01x01, yarrboard:T44001, F.Cu at (-51.7, 22.1)
- added J15: Conn_01x01, yarrboard:T44001, F.Cu at (-51.7, -12.2)
- added J16: Conn_01x02, Connector_JST:JST_PH_B2B-PH-K_1x02_P2.00mm_Vertical, F.Cu at (-65.0, 60.0)
- added J17: Conn_01x02, Connector_JST:JST_PH_B2B-PH-K_1x02_P2.00mm_Vertical, F.Cu at (-65.0, 51.5)
- added J18: Conn_01x02, Connector_JST:JST_PH_B2B-PH-K_1x02_P2.00mm_Vertical, F.Cu at (-55.0, 60.0)
- added J19: Conn_01x02, Connector_JST:JST_PH_B2B-PH-K_1x02_P2.00mm_Vertical, F.Cu at (-55.0, 51.5)
- added JP3: SolderJumper_2_Open, Jumper:SolderJumper-2_P1.3mm_Open_RoundedPad1.0x1.5mm, F.Cu at (-44.1, 40.3)
- added JP4: SolderJumper_2_Open, Jumper:SolderJumper-2_P1.3mm_Open_RoundedPad1.0x1.5mm, F.Cu at (-28.2, 31.4)
- added JP5: SolderJumper_2_Open, Jumper:SolderJumper-2_P1.3mm_Open_RoundedPad1.0x1.5mm, F.Cu at (-28.2, 35.0)
- added Q35: 2N7002, Package_TO_SOT_SMD:SOT-23, F.Cu at (-65.5, -27.7)
- added Q36: BC846, Package_TO_SOT_SMD:SOT-23, F.Cu at (-65.5, -23.1)
- added Q37: BC856, Package_TO_SOT_SMD:SOT-23, F.Cu at (-65.5, -18.5)
- added Q38: IPB110P06LM, Package_TO_SOT_SMD:TO-263-2, F.Cu at (-79.7, -24.0)
- added Q39: 2N7002, Package_TO_SOT_SMD:SOT-23, F.Cu at (-31.3, 6.53)
- added Q40: BC846, Package_TO_SOT_SMD:SOT-23, F.Cu at (-31.3, 11.2)
- added Q41: BC856, Package_TO_SOT_SMD:SOT-23, F.Cu at (-31.3, 15.8)
- added Q42: IPB110P06LM, Package_TO_SOT_SMD:TO-263-2, F.Cu at (-45.5, 10.3)
- added Q43: 2N7002, Package_TO_SOT_SMD:SOT-23, F.Cu at (-65.5, 6.53)
- added Q44: BC846, Package_TO_SOT_SMD:SOT-23, F.Cu at (-65.5, 11.2)
- added Q45: BC856, Package_TO_SOT_SMD:SOT-23, F.Cu at (-65.5, 15.8)
- added Q46: IPB110P06LM, Package_TO_SOT_SMD:TO-263-2, F.Cu at (-79.7, 10.3)
- added Q47: 2N7002, Package_TO_SOT_SMD:SOT-23, F.Cu at (-31.3, -27.7)
- added Q48: BC846, Package_TO_SOT_SMD:SOT-23, F.Cu at (-31.3, -23.1)
- added Q49: BC856, Package_TO_SOT_SMD:SOT-23, F.Cu at (-31.3, -18.5)
- added Q50: IPB110P06LM, Package_TO_SOT_SMD:TO-263-2, F.Cu at (-45.5, -24.0)
- added R100: 0, Resistor_SMD:R_0805_2012Metric_Pad1.20x1.40mm_HandSolder, F.Cu at (-19.7, 16.2)
- added R101: 0, Resistor_SMD:R_0805_2012Metric_Pad1.20x1.40mm_HandSolder, F.Cu at (-19.7, 19.1)
- added R102: 165 0.1%, Resistor_SMD:R_0805_2012Metric_Pad1.20x1.40mm_HandSolder, F.Cu at (-19.7, 22.1)
- added R103: 0, Resistor_SMD:R_0805_2012Metric_Pad1.20x1.40mm_HandSolder, F.Cu at (-74.5, 31.1)
- added R104: 0, Resistor_SMD:R_0805_2012Metric_Pad1.20x1.40mm_HandSolder, F.Cu at (-74.5, 34.1)
- added R105: 165 0.1%, Resistor_SMD:R_0805_2012Metric_Pad1.20x1.40mm_HandSolder, F.Cu at (-74.5, 37.0)
- added R106: 0, Resistor_SMD:R_0805_2012Metric_Pad1.20x1.40mm_HandSolder, F.Cu at (-81.2, 31.1)
- added R107: 0, Resistor_SMD:R_0805_2012Metric_Pad1.20x1.40mm_HandSolder, F.Cu at (-81.2, 34.1)
- added R108: 165 0.1%, Resistor_SMD:R_0805_2012Metric_Pad1.20x1.40mm_HandSolder, F.Cu at (-81.2, 37.0)
- added R109: 10k, Resistor_SMD:R_0805_2012Metric_Pad1.20x1.40mm_HandSolder, F.Cu at (-14.9, 1.53)
- added R110: 10k, Resistor_SMD:R_0805_2012Metric_Pad1.20x1.40mm_HandSolder, F.Cu at (-16.9, 35.8)
- added R111: 10k, Resistor_SMD:R_0805_2012Metric_Pad1.20x1.40mm_HandSolder, F.Cu at (-14.9, 11.2)
- added R12: 300K, Resistor_SMD:R_0805_2012Metric_Pad1.20x1.40mm_HandSolder, F.Cu at (-19.7, -13.7)
- added R13: 22K, Resistor_SMD:R_0805_2012Metric_Pad1.20x1.40mm_HandSolder, F.Cu at (-19.7, -10.7)
- added R19: 300K, Resistor_SMD:R_0805_2012Metric_Pad1.20x1.40mm_HandSolder, F.Cu at (-61.0, 31.1)
- added R20: 22K, Resistor_SMD:R_0805_2012Metric_Pad1.20x1.40mm_HandSolder, F.Cu at (-61.0, 34.1)
- added R26: 300K, Resistor_SMD:R_0805_2012Metric_Pad1.20x1.40mm_HandSolder, F.Cu at (-19.7, -37.4)
- added R27: 22K, Resistor_SMD:R_0805_2012Metric_Pad1.20x1.40mm_HandSolder, F.Cu at (-19.7, -34.4)
- added R40: 300K, Resistor_SMD:R_0805_2012Metric_Pad1.20x1.40mm_HandSolder, F.Cu at (-67.8, 39.0)
- added R47: 300K, Resistor_SMD:R_0805_2012Metric_Pad1.20x1.40mm_HandSolder, F.Cu at (-61.0, 39.0)
- added R48: 22K, Resistor_SMD:R_0805_2012Metric_Pad1.20x1.40mm_HandSolder, F.Cu at (-61.0, 42.0)
- added R5: 300K, Resistor_SMD:R_0805_2012Metric_Pad1.20x1.40mm_HandSolder, F.Cu at (-67.8, 31.1)
- added R54: 300K, Resistor_SMD:R_0805_2012Metric_Pad1.20x1.40mm_HandSolder, F.Cu at (-19.7, -21.6)
- added R55: 22K, Resistor_SMD:R_0805_2012Metric_Pad1.20x1.40mm_HandSolder, F.Cu at (-19.7, -18.6)
- added R6: 22K, Resistor_SMD:R_0805_2012Metric_Pad1.20x1.40mm_HandSolder, F.Cu at (-67.8, 34.1)
- added R63: 10k, Resistor_SMD:R_0805_2012Metric_Pad1.20x1.40mm_HandSolder, F.Cu at (-43.9, 31.1)
- added R64: 300K 0.1%, Resistor_SMD:R_0805_2012Metric_Pad1.20x1.40mm_HandSolder, F.Cu at (-43.9, 34.1)
- added R65: 22K 0.1%, Resistor_SMD:R_0805_2012Metric_Pad1.20x1.40mm_HandSolder, F.Cu at (-43.9, 37.0)
- added R69: 1k, Resistor_SMD:R_0805_2012Metric_Pad1.20x1.40mm_HandSolder, F.Cu at (-70.3, -28.7)
- added R70: 220R, Resistor_SMD:R_0805_2012Metric_Pad1.20x1.40mm_HandSolder, F.Cu at (-70.3, -25.7)
- added R71: 27k, Resistor_SMD:R_0805_2012Metric_Pad1.20x1.40mm_HandSolder, F.Cu at (-70.3, -22.8)
- added R72: 4.7k, Resistor_SMD:R_0805_2012Metric_Pad1.20x1.40mm_HandSolder, F.Cu at (-70.3, -19.8)
- added R73: 300K, Resistor_SMD:R_0805_2012Metric_Pad1.20x1.40mm_HandSolder, F.Cu at (-70.3, -16.9)
- added R74: 22K, Resistor_SMD:R_0805_2012Metric_Pad1.20x1.40mm_HandSolder, F.Cu at (-70.3, -13.9)
- added R75: 1k, Resistor_SMD:R_0805_2012Metric_Pad1.20x1.40mm_HandSolder, F.Cu at (-70.3, -11.0)
- added R76: 1k, Resistor_SMD:R_0805_2012Metric_Pad1.20x1.40mm_HandSolder, F.Cu at (-36.1, 5.60)
- added R77: 220R, Resistor_SMD:R_0805_2012Metric_Pad1.20x1.40mm_HandSolder, F.Cu at (-36.1, 8.55)
- added R78: 27k, Resistor_SMD:R_0805_2012Metric_Pad1.20x1.40mm_HandSolder, F.Cu at (-36.1, 11.5)
- added R79: 4.7k, Resistor_SMD:R_0805_2012Metric_Pad1.20x1.40mm_HandSolder, F.Cu at (-36.1, 14.4)
- added R80: 300K, Resistor_SMD:R_0805_2012Metric_Pad1.20x1.40mm_HandSolder, F.Cu at (-36.1, 17.4)
- added R81: 22K, Resistor_SMD:R_0805_2012Metric_Pad1.20x1.40mm_HandSolder, F.Cu at (-36.1, 20.4)
- added R82: 1k, Resistor_SMD:R_0805_2012Metric_Pad1.20x1.40mm_HandSolder, F.Cu at (-36.1, 23.3)
- added R83: 1k, Resistor_SMD:R_0805_2012Metric_Pad1.20x1.40mm_HandSolder, F.Cu at (-70.3, 5.60)
- added R84: 220R, Resistor_SMD:R_0805_2012Metric_Pad1.20x1.40mm_HandSolder, F.Cu at (-70.3, 8.55)
- added R85: 27k, Resistor_SMD:R_0805_2012Metric_Pad1.20x1.40mm_HandSolder, F.Cu at (-70.3, 11.5)
- added R86: 4.7k, Resistor_SMD:R_0805_2012Metric_Pad1.20x1.40mm_HandSolder, F.Cu at (-70.3, 14.4)
- added R87: 300K, Resistor_SMD:R_0805_2012Metric_Pad1.20x1.40mm_HandSolder, F.Cu at (-70.3, 17.4)
- added R88: 22K, Resistor_SMD:R_0805_2012Metric_Pad1.20x1.40mm_HandSolder, F.Cu at (-70.3, 20.4)
- added R89: 1k, Resistor_SMD:R_0805_2012Metric_Pad1.20x1.40mm_HandSolder, F.Cu at (-70.3, 23.3)
- added R90: 1k, Resistor_SMD:R_0805_2012Metric_Pad1.20x1.40mm_HandSolder, F.Cu at (-36.1, -28.7)
- added R91: 220R, Resistor_SMD:R_0805_2012Metric_Pad1.20x1.40mm_HandSolder, F.Cu at (-36.1, -25.7)
- added R92: 27k, Resistor_SMD:R_0805_2012Metric_Pad1.20x1.40mm_HandSolder, F.Cu at (-36.1, -22.8)
- added R93: 4.7k, Resistor_SMD:R_0805_2012Metric_Pad1.20x1.40mm_HandSolder, F.Cu at (-36.1, -19.8)
- added R94: 300K, Resistor_SMD:R_0805_2012Metric_Pad1.20x1.40mm_HandSolder, F.Cu at (-36.1, -16.9)
- added R95: 22K, Resistor_SMD:R_0805_2012Metric_Pad1.20x1.40mm_HandSolder, F.Cu at (-36.1, -13.9)
- added R96: 1k, Resistor_SMD:R_0805_2012Metric_Pad1.20x1.40mm_HandSolder, F.Cu at (-36.1, -11.0)
- added R97: 0, Resistor_SMD:R_0805_2012Metric_Pad1.20x1.40mm_HandSolder, F.Cu at (-88.0, 31.1)
- added R98: 0, Resistor_SMD:R_0805_2012Metric_Pad1.20x1.40mm_HandSolder, F.Cu at (-88.0, 34.1)
- added R99: 165 0.1%, Resistor_SMD:R_0805_2012Metric_Pad1.20x1.40mm_HandSolder, F.Cu at (-88.0, 37.0)
- added U11: MCP1502-33, Package_TO_SOT_SMD:SOT-23-6, F.Cu at (-48.8, 32.1)
- added U12: MCP3425A0T-ECH, Package_TO_SOT_SMD:SOT-23-6, F.Cu at (-48.8, 36.7)
- added U14: MCP3564R, Package_SO:TSSOP-20_4.4x6.5mm_P0.65mm, F.Cu at (-34.8, 33.7)
- added U16: ACS725xLCTR-20AU, yarrboard:ACS7XX, F.Cu at (-29.6, 21.7)
- added U17: ACS725xLCTR-20AU, yarrboard:ACS7XX, F.Cu at (-63.7, 21.7)
- added U18: ACS725xLCTR-20AU, yarrboard:ACS7XX, F.Cu at (-29.6, -12.6)
- added U19: ADS1015IDGS, Package_SO:TSSOP-10_3x3mm_P0.5mm, F.Cu at (-18.6, -2.27)
- added U20: ADS1015IDGS, Package_SO:TSSOP-10_3x3mm_P0.5mm, F.Cu at (-20.6, 32.0)
- added U21: ADS1015IDGS, Package_SO:TSSOP-10_3x3mm_P0.5mm, F.Cu at (-18.6, 7.39)
- C29: value 100nF -> 10uF
- C48: value 10uF -> 4.7nF
- D39: value BAT54S -> SS16; footprint Package_TO_SOT_SMD:SOT-23 -> Diode_SMD:D_SMA
- J14: value N2K -> Conn_01x01; footprint Connector_PinHeader_2.54mm:PinHeader_1x04_P2.54mm_Vertical -> yarrboard:T44001
- R33: value 300K 0.1% -> 300K
- R34: value 22K 0.1% -> 22K
- R41: value 10k -> 22K
- U15: value MCP3425A0T-ECH -> ACS725xLCTR-20AU; footprint Package_TO_SOT_SMD:SOT-23-6 -> yarrboard:ACS7XX
- moved D39 190.0 mm to (-77.2, -15.5)
- moved U15 174.2 mm to (-63.7, -12.6), turned to 0 degrees
- moved J7 171.9 mm to (165.0, 129.0)
- moved J8 169.0 mm to (177.0, 129.0)
- moved J6 167.2 mm to (153.0, 129.0)
- moved R34 160.8 mm to (-19.7, -26.5), turned to 0 degrees
- moved R33 160.1 mm to (-19.7, -29.5), turned to 0 degrees
- moved C48 151.4 mm to (-26.5, -22.6), turned to 0 degrees
- moved J14 149.7 mm to (-85.8, 22.1), turned to 0 degrees
- moved R41 147.2 mm to (-67.8, 42.0)
- moved C29 144.8 mm to (-53.8, 37.2), turned to 0 degrees
- moved J5 139.0 mm to (141.0, 129.0)
- moved C28 137.6 mm to (-53.8, 34.2), turned to 0 degrees
- moved J3 137.4 mm to (117.0, 129.0)
- moved J4 133.5 mm to (129.0, 129.0)
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- renumbered C3 to C1, C12 to C10, C13 to C11, C14 to C12, C15 to C13, C16 to C14, C17 to C15, C18 to C16, C19 to C17, C20 to C18, C21 to C19, C4 to C2, C22 to C20, C23 to C21, C24 to C22, C25 to C23, C26 to C24, C49 to C25, C2 to C27, C5 to C3, C1 to C30, C43 to C32, C44 to C33, C45 to C34, C47 to C35, C6 to C4, C7 to C5, C8 to C6, C9 to C7, C10 to C8, C11 to C9, D2 to D1, D5 to D10, D21 to D11, D13 to D12, D6 to D13, D22 to D14, D14 to D15, D7 to D16, D23 to D17, D15 to D18, D8 to D19, D18 to D2, D24 to D20, D16 to D21, D9 to D22, D25 to D23, D17 to D24, D34 to D25, D36 to D26, D35 to D27, D37 to D28, D1 to D29, D10 to D3, D27 to D30, D28 to D31, D38 to D33, D33 to D35, D26 to D36, D3 to D4, D19 to D5, D11 to D6, D4 to D7, D20 to D8, D12 to D9, FB7 to FB1, J3 to J10, J4 to J11, J5 to J3, J6 to J4, J7 to J5, J8 to J6, J9 to J7, J10 to J8, J13 to J9, JP2 to JP1, JP3 to JP2, M2 to M1, M1 to M2, Q25 to Q10, Q26 to Q11, Q6 to Q12, Q7 to Q13, Q27 to Q14, Q28 to Q15, Q8 to Q16, Q9 to Q17, Q29 to Q18, Q30 to Q19, Q21 to Q2, Q10 to Q20, Q11 to Q21, Q31 to Q22, Q32 to Q23, Q12 to Q24, Q13 to Q25, Q33 to Q26, Q34 to Q27, Q14 to Q28, Q15 to Q29, Q22 to Q3, Q35 to Q30, Q36 to Q31, Q16 to Q32, Q17 to Q33, Q18 to Q34, Q2 to Q4, Q3 to Q5, Q23 to Q6, Q24 to Q7, Q4 to Q8, Q5 to Q9, R7 to R10, R8 to R11, R48 to R14, R9 to R15, R10 to R16, R11 to R17, R12 to R18, R49 to R21, R13 to R22, R14 to R23, R15 to R24, R16 to R25, R50 to R28, R17 to R29, R18 to R30, R19 to R31, R20 to R32, R51 to R35, R21 to R36, R22 to R37, R23 to R38, R24 to R39, R52 to R42, R25 to R43, R26 to R44, R27 to R45, R28 to R46, R53 to R49, R29 to R50, R30 to R51, R31 to R52, R32 to R53, R54 to R56, R43 to R57, R36 to R58, R44 to R59, R35 to R60, R40 to R61, R42 to R62, R39 to R66, R37 to R67, R38 to R68, R47 to R7, R5 to R8, R6 to R9, U3 to U10, U4 to U13, U5 to U2, U6 to U3, U7 to U4, U8 to U5, U9 to U6, U10 to U7, U11 to U8, U12 to U9
Connections:
- net /ADC/A0 renamed /CHANNEL 0/CURRENT_ADC
- net /ADC/A1 renamed /CHANNEL 1/CURRENT_ADC
- net /ADC/A2 renamed /CHANNEL 2/CURRENT_ADC
- net /ADC/A3 renamed /CHANNEL 3/CURRENT_ADC
- net /ADC/A4 renamed /CHANNEL 4/CURRENT_ADC
- net /ADC/A5 renamed /CHANNEL 5/CURRENT_ADC
- net /ADC/A6 renamed /CHANNEL 6/CURRENT_ADC
- net /ADC/A7 renamed /CHANNEL 7/CURRENT_ADC
- C28 pad 1: +3.3V -> Net-(C28-Pad1)
- C29 pad 1: ESP32_5V -> +3.3V
- C48 pad 1: +3.3V -> /CHANNEL 11/CURRENT_ADC
- D15 pad 1: Net-(D14-K) (its old number) -> Net-(D15-K)
- D39 pad 1: GNDA -> Net-(D39-K)
- D39 pad 2: +3.3V -> GNDPWR
- F5 pad 3: Net-(D14-K) (its old number) -> Net-(D15-K)
- J14 pad 1: CAN_RX -> Net-(D45-K)
- J5 pad 1: Net-(D14-K) (its old number) -> Net-(D15-K)
- R33 pad 1: Net-(D39-COM) -> VOLT4
- R33 pad 2: +24V -> Net-(D15-K)
- R34 pad 1: GNDA -> GNDPWR
- R34 pad 2: Net-(D39-COM) -> VOLT4
- R41 pad 1: Net-(C30-Pad1) -> GNDPWR
- R41 pad 2: REF_3V3 -> VOLT5
- U1 pad 10: CAN_TX -> FAN_TACH1
- U1 pad 11: CAN_RX -> ADC1_CS
- U1 pad 16: SS -> ADC0_SS
- U1 pad 20: unconnected-(U1-GPIO14-Pad20) -> /CHANNEL 11/PWM
- U1 pad 27: FAN_TACH1 -> /CHANNEL 10/PWM
- U1 pad 28: FAN_PWM1 -> /CHANNEL 9/PWM
- U1 pad 29: FAN_MOSFET1 -> /CHANNEL 8/PWM
- U1 pad 8: unconnected-(U1-GPIO15-Pad8) -> FAN_MOSFET1
- U1 pad 9: unconnected-(U1-GPIO16-Pad9) -> FAN_PWM1
- U10 pad 13: SS -> ADC0_CS
- U15 pad 1: Net-(D39-COM) -> Net-(Q38-D)
- U15 pad 2: GNDA -> Net-(Q38-D)
- U15 pad 3: SCL -> Net-(D39-K)
- U15 pad 4: SDA -> Net-(D39-K)
- U15 pad 5: +3.3V -> GNDA
- U15 pad 6: GNDA -> Net-(U15-FILTER)
- U6 pad 3: Net-(D14-K) (its old number) -> Net-(D15-K)
- U6 pad 4: Net-(D14-K) (its old number) -> Net-(D15-K)
Routing:
- net Net-(D3-K): track 166.1 -> 0.00 mm
- net /CHANNEL 7/PWM: track 156.0 -> 0.00 mm
- net +3.3V: track 159.5 -> 4.05 mm
- net /CHANNEL 6/CURRENT_ADC: track 146.7 -> 0.00 mm
- net /CHANNEL 6/PWM: track 136.4 -> 0.00 mm
- net /CHANNEL 5/CURRENT_ADC: track 127.4 -> 0.00 mm
- net /CHANNEL 5/PWM: track 116.9 -> 0.00 mm
- net /CHANNEL 4/CURRENT_ADC: track 108.1 -> 0.00 mm
- net /CHANNEL 4/PWM: track 97.3 -> 0.00 mm
- net /CHANNEL 3/CURRENT_ADC: track 89.0 -> 0.00 mm
- net /CHANNEL 3/PWM: track 77.9 -> 0.00 mm
- net /CHANNEL 2/CURRENT_ADC: track 69.8 -> 0.00 mm
- net FAN_TACH1: track 60.1 -> 0.00 mm
- net /CHANNEL 2/PWM: track 58.7 -> 0.00 mm
- net /CHANNEL 1/CURRENT_ADC: track 50.4 -> 0.00 mm
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- added copper zone on B.Cu, net Net-(D11-K)
- added copper zone on B.Cu, net Net-(D12-K)
- added copper zone on B.Cu, net Net-(D14-K)
- added copper zone on B.Cu, net Net-(D15-K)
- added copper zone on F.Cu, net Net-(D15-K)
- added copper zone on B.Cu, net Net-(D17-K)
- added copper zone on B.Cu, net Net-(D21-K)
- added copper zone on B.Cu, net Net-(D3-K)
- removed copper zone on F.Cu, net Net-(D14-K) (its old number)
- removed copper zone on F.Cu, net Net-(D2-K)
- removed copper zone on F.Cu, net Net-(D6-K)
- removed copper zone on F.Cu, net Net-(D8-K)
- removed copper zone on F.Cu, net Net-(D9-K)
- removed copper zone on B.Cu, net Net-(Q12-D)
- removed copper zone on B.Cu, net Net-(Q16-D)
- removed copper zone on B.Cu, net Net-(Q20-D)
- removed copper zone on B.Cu, net Net-(Q24-D)
- removed copper zone on F.Cu, net Net-(Q24-D)
- removed copper zone on B.Cu, net Net-(Q28-D)
- removed copper zone on B.Cu, net Net-(Q32-D)
- removed copper zone on F.Cu, net Net-(Q32-D)
- removed copper zone on B.Cu, net Net-(Q4-D)
- removed copper zone on B.Cu, net Net-(Q8-D)
Other:
- board size 184.5 x 137 mm -> 141 x 269 mm
- board text added: "CH0"
- board text removed: "CH0-"
- board text removed: "CH1+"
- board text removed: "CH1-"
- board text removed: "CH2+"
- board text removed: "CH2-"
- board text removed: "CH3+"
- board text removed: "CH3-"
- board text removed: "CH4+"
- board text removed: "CH4-"
- board text removed: "CH5+"
- board text removed: "CH5-"
- board text removed: "CH6+"
- board text removed: "CH6-"
- board text removed: "CH7+"
- board text removed: "CH7-"
