File: 8ch-mosfet/voltage_adc.kicad_sch (KiCad schematic)
At the start: 3 parts, among them U20 ADS1015IDGS

Commit message: component layout looking crispy.
Parts:
- renumbered C49 to C50, R109 to R110
Changed lines of the file:
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@@
 		(on_board yes)
 		(dnp no)
-		(property "Reference" "C49"
+		(property "Reference" "C50"
 			(at 170.18 82.5563 0)
 			(effects
@@
 		(dnp no)
 		(fields_autoplaced yes)
-		(property "Reference" "R109"
+		(property "Reference" "R110"
 			(at 160.02 82.55 0)
 			(effects
@@
 		(on_board yes)
 		(dnp no)
-		(property "Reference" "#PWR0106"
+		(property "Reference" "#PWR0107"
 			(at 138.43 115.57 0)
 			(effects
@@
 			(project "8ch-mosfet"
 				(path "/c83c6236-96e9-46ad-9d7a-9e2efa4a7966/a6260305-24e3-4714-b441-a7a157c17bd9"
-					(reference "#PWR0108")
-					(unit 1)
-				)
-				(path "/c83c6236-96e9-46ad-9d7a-9e2efa4a7966/bb9dea8b-8412-49bc-950d-dce57727bcd2"
-					(reference "#PWR0106")
-					(unit 1)
-				)
-				(path "/c83c6236-96e9-46ad-9d7a-9e2efa4a7966/efce81b0-0da6-4cc8-a856-27910d231a7d"
-					(reference "#PWR0110")
+					(reference "#PWR0107")
+					(unit 1)
+				)
+				(path "/c83c6236-96e9-46ad-9d7a-9e2efa4a7966/bb9dea8b-8412-49bc-950d-dce57727bcd2"
+					(reference "#PWR0105")
+					(unit 1)
+				)
+				(path "/c83c6236-96e9-46ad-9d7a-9e2efa4a7966/efce81b0-0da6-4cc8-a856-27910d231a7d"
+					(reference "#PWR0109")
 					(unit 1)
 				)
@@
 		(dnp no)
 		(fields_autoplaced yes)
-		(property "Reference" "#PWR0105"
+		(property "Reference" "#PWR0106"
 			(at 138.43 80.01 0)
 			(effects
@@
 			(project "8ch-mosfet"
 				(path "/c83c6236-96e9-46ad-9d7a-9e2efa4a7966/a6260305-24e3-4714-b441-a7a157c17bd9"
-					(reference "#PWR0107")
-					(unit 1)
-				)
-				(path "/c83c6236-96e9-46ad-9d7a-9e2efa4a7966/bb9dea8b-8412-49bc-950d-dce57727bcd2"
-					(reference "#PWR0105")
-					(unit 1)
-				)
-				(path "/c83c6236-96e9-46ad-9d7a-9e2efa4a7966/efce81b0-0da6-4cc8-a856-27910d231a7d"
-					(reference "#PWR0109")
-					(unit 1)
-				)
+					(reference "#PWR0106")
+					(unit 1)
+				)
+				(path "/c83c6236-96e9-46ad-9d7a-9e2efa4a7966/bb9dea8b-8412-49bc-950d-dce57727bcd2"
+					(reference "#PWR0104")
+					(unit 1)
+				)
+				(path "/c83c6236-96e9-46ad-9d7a-9e2efa4a7966/efce81b0-0da6-4cc8-a856-27910d231a7d"
+					(reference "#PWR0108")
+					(unit 1)
+				)
