File: 8ch-mosfet/adc.kicad_sch (KiCad schematic)
At the start: 13 parts, among them U13 MCP1502-33, U15 MCP3425A0T-ECH, U2 MCP3208

Commit message: changed to MCP3564
Parts:
- removed U2: MCP3208, Package_SO:SOIC-16_3.9x9.9mm_P1.27mm, symbol Analog_ADC:MCP3208
- added JP2, JP3: SolderJumper_2_Open, Jumper:SolderJumper-2_P1.3mm_Open_RoundedPad1.0x1.5mm, symbol Jumper:SolderJumper_2_Open
- added U3: MCP3564R, Package_SO:TSSOP-20_4.4x6.5mm_P0.65mm, symbol yarrboard:MCP3564R
- renumbered C3 to C28, C3 to C29, C3 to C30, C3 to C48, C3 to C49, R33 to R41
Connections:
- net +3.3V: now also C49.1, JP3.1 (A), U3.20 (DVDD)
- net A0: now also U3.5 (CH0)
- net A1: now also U3.6 (CH1)
- net A2: now also U3.7 (CH2)
- net A3: now also U3.8 (CH3)
- net A4: now also U3.9 (CH4)
- net A5: now also U3.10 (CH5)
- net A6: now also U3.11 (CH6)
- net A7: now also U3.12 (CH7)
- net GNDA: now also U3.2 (AGND), U3.3 (VREF-); no longer C49.2
- net GNDD: now also C49.2, U3.19 (DGND)
- net MISO: now also U3.16 (SDO)
- net MOSI: now also U3.15 (SDI)
- net REF_3V3: now also JP2.2 (B), U3.4 (VREF+); no longer C49.1
- net SCK: now also U3.14 (SCK)
- net SS: now also U3.13 (~{CS})
- new net: JP2.1 (A), JP3.2 (B), U3.1 (AVDD)
Other:
- moved on the sheet: C49

Commit message: big update - 12ch, volt adc, senders, etc.
Parts:
- removed C28, C29, C30: 100nF, Capacitor_SMD:C_0805_2012Metric_Pad1.18x1.45mm_HandSolder, symbol Device:C_Small
- removed C48: 10uF, Capacitor_SMD:C_0805_2012Metric_Pad1.18x1.45mm_HandSolder, symbol Device:C_Small
- removed D39: BAT54S, Package_TO_SOT_SMD:SOT-23, symbol Diode:BAT54S
- removed JP1: SolderJumper_2_Open, Jumper:SolderJumper-2_P1.3mm_Open_RoundedPad1.0x1.5mm, symbol Jumper:SolderJumper_2_Open
- removed R33: 300K 0.1%, Resistor_SMD:R_0805_2012Metric_Pad1.20x1.40mm_HandSolder, symbol Device:R_Small_US
- removed R34: 22K 0.1%, Resistor_SMD:R_0805_2012Metric_Pad1.20x1.40mm_HandSolder, symbol Device:R_Small_US
- removed R41: 10k, Resistor_SMD:R_0805_2012Metric_Pad1.20x1.40mm_HandSolder, symbol Device:R_Small_US
- removed U13: MCP1502-33, Package_TO_SOT_SMD:SOT-23-6, symbol Reference_Voltage:MCP1501-30xCH
- removed U15: MCP3425A0T-ECH, Package_TO_SOT_SMD:SOT-23-6, symbol Analog_ADC:MCP3425A0T-ECH
- renumbered C49 to C36, JP2 to JP4, JP3 to JP5, U3 to U14
Connections:
- net SS renamed ~{CS}
Other:
- note removed: "Bus Voltage Circuit"
- note removed: "Reference Voltage Circuit"
- moved on the sheet: C36, JP4, JP5, U14

Commit message: more layout work.  going to be a beast.
Parts:
- removed JP4, JP5: SolderJumper_2_Open, Jumper:SolderJumper-2_P1.3mm_Open_RoundedPad1.0x1.5mm, symbol Jumper:SolderJumper_2_Open
- added C52: 100nF, Capacitor_SMD:C_0805_2012Metric_Pad1.18x1.45mm_HandSolder, symbol Device:C_Small
Connections:
- net GNDA: now also C52.2
- net REF_3V3: now also U14.1 (AVDD), C52.1
Other:
- moved on the sheet: C36, U14
